File: electrode-pcb/cortipod-electrode-panel.kicad_pcb (KiCad board)
At the start: 2 copper layers, 88 x 66 mm, 48 parts

Commit message: Fix panelized PCB for JLCPCB V-cut: add 3mm breakaway rails (88x72mm)
JLCPCB rejected the 88x66mm panel (below 70x70mm V-cut minimum) and
required minimum 3mm edge rails. Added 3mm top/bottom breakaway rails
bringing the panel to 88x72mm. Cell positions are unchanged in absolute
coordinates so in-production stencils remain compatible.

Co-Authored-By: Claude Opus 4.6 (1M context) <noreply@anthropic.com>
Other:
- board size 88 x 66 mm -> 88 x 72 mm
- board text added: "CortiPod Electrode Panel 4x3 = 12 cells + rails - V-SCORE at marked lines"
- board text removed: "CortiPod Electrode Panel 4x3 = 12 cells - V-SCORE at marked lines"
